File: MRCS-cpNode.brd (EAGLE design)
At the start: 99.8 x 68.8 mm, 50 parts, among them CON1 0.100, CON2 0.100, CON3 0.100, CON4 0.100, J1 0.100, J2 0.100, P1 CA CC, U1 MAX3465CPD, U2 NE555P

Commit message: silk and trace cleanup
Parts:
- moved RS485-1 2.54 mm to (11.4, 44.5)
- moved RS485-2 2.54 mm to (33.0, 44.5)
- moved RS485-3 2.54 mm to (11.4, 54.0)
- moved RS485-4 2.54 mm to (31.8, 54.0)
- moved IO1 1.91 mm to (83.8, 50.8)
- moved IO2 1.91 mm to (63.5, 50.8)
- moved IO3 1.91 mm to (83.8, 40.6)
- moved IO4 1.91 mm to (63.5, 40.6)
- moved SJ1 1.91 mm to (83.8, 46.4)
- moved SJ10 1.91 mm to (61.0, 46.4)
- moved SJ11 1.91 mm to (58.4, 46.4)
- moved SJ12 1.91 mm to (55.9, 46.4)
- moved SJ13 1.91 mm to (53.3, 46.4)
- moved SJ14 1.91 mm to (50.8, 46.4)
- moved SJ15 1.91 mm to (48.3, 46.4)
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Routing:
- net T+: track 57.5 -> 54.9 mm
- net T-: track 61.7 -> 59.1 mm
- net R-: track 62.4 -> 59.9 mm
- net R+: track 64.8 -> 62.2 mm
- net O13: track 27.0 -> 28.9 mm
- net O8: track 15.5 -> 17.4 mm
- net O6: track 15.5 -> 17.4 mm
- net O7: track 15.8 -> 17.7 mm
- net O5: track 15.8 -> 17.7 mm
- net O4: track 16.1 -> 18.0 mm
- net O3: track 16.3 -> 18.2 mm
- net O2: track 16.1 -> 18.0 mm
- net O15: track 27.4 -> 29.3 mm
- net O1: track 16.3 -> 18.2 mm
- net D9: track 15.0 -> 13.1 mm
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Other:
- board text added: "2021-06"
- board text added: "v2.7"
- board text removed: "2020-01"
- board text removed: "v2.6"

Commit message: silk cleanuo
Parts:
- moved U$3 59.1 mm to (21.6, 21.6)
- moved U$2 33.0 mm to (75.6, 17.8)
- moved TX 1.27 mm to (21.6, 36.8), turned to 180 degrees
Routing:
- net GND: track 45.4 -> 37.8 mm
- net N$29: track 2.54 -> 5.61 mm
- net TX: track 122.2 -> 121.5 mm
Other:
- board text added: "5v"
- board text added: "BBLeo"
- board text added: "MRCS Control Point Node"
- board text added: "SCL"
- board text added: "SDA"
- board text removed: "Control Point Node"
